File: YRM1001/YRM1001.kicad_sch (KiCad schematic)
At the start: 11 parts, among them J1 picoblade, J2 Conn_01x05

Commit message: Add files via upload
updated board version to 1.2:
- changed ICSP from 10 pin header to 6 pin header. 10 pin ICSP connections can be done with a 6 to 10 pin adapter cable.
- changed name on board to UHF | RFID | SAM, removing '1/2 nard' from the name for clarity on what the board is and does.
- removed header that was meant to hard-connect the UHF module to the board: it is not used for communication with the board after all. 
- updated the QR codes designs for better machine readability
- various routing improvements.

schematics:
- changed ICSP from 10 pin header to 6 pin header

other:
reverse-engineered the YRM1001 and YRM200 boards to have them in Kicad. Measurements should be close enough for OKing designs using those modules.
Parts:
- added H1, H2, H3, H4: MountingHole_Pad, MountingHole:MountingHole_2.2mm_M2_ISO7380_Pad, symbol Mechanical:MountingHole_Pad
Connections:
- net GND: now also H1.1, H2.1, H3.1, H4.1
Changed lines of the file:
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@@
 (kicad_sch (version 20230121) (generator eeschema)
   (paper "A4")
+  (junction (at 133.35 97.79) (diameter 0) (color 0 0 0 0)
+  )
   (junction (at 77.47 128.27) (diameter 0) (color 0 0 0 0)
   )
@@
   (junction (at 74.93 95.25) (diameter 0) (color 0 0 0 0)
   )
+  (junction (at 128.27 97.79) (diameter 0) (color 0 0 0 0)
+  )
   (junction (at 81.28 158.75) (diameter 0) (color 0 0 0 0)
   )
   (junction (at 57.15 158.75) (diameter 0) (color 0 0 0 0)
+  )
+  (junction (at 123.19 97.79) (diameter 0) (color 0 0 0 0)
   )
   (no_connect (at 73.66 158.75))
@@
     (stroke (width 0) (type default))
   )
+  (wire (pts (xy 128.27 97.79) (xy 133.35 97.79))
+    (stroke (width 0) (type default))
+  )
   (wire (pts (xy 95.25 128.27) (xy 96.52 128.27))
     (stroke (width 0) (type default))
@@
     (stroke (width 0) (type default))
   )
+  (wire (pts (xy 133.35 97.79) (xy 138.43 97.79))
+    (stroke (width 0) (type default))
+  )
   (wire (pts (xy 57.15 134.62) (xy 57.15 147.32))
     (stroke (width 0) (type default))
@@
   )
   (wire (pts (xy 57.15 158.75) (xy 57.15 161.29))
+    (stroke (width 0) (type default))
+  )
+  (wire (pts (xy 123.19 97.79) (xy 128.27 97.79))
     (stroke (width 0) (type default))
   )
@@
         (path "/d8d0a45f-1f46-4ba4-9944-4b3c9d150d73"
           (reference "#PWR02") (unit 1)
+        )
+      )
+    )
+  )
+  (symbol (lib_id "Mechanical:MountingHole_Pad") (at 128.27 95.25 0) (unit 1)
+    (in_bom yes) (on_board yes) (dnp no)
+    (property "Reference" "H2" (at 127 90.17 0)
+      (effects (font (size 1.27 1.27)) (justify left))
+    )
+    (property "Value" "MountingHole_Pad" (at 120.4892 100.33 0)
+      (effects (font (size 1.27 1.27)) (justify left) hide)
+    )
+    (property "Footprint" "MountingHole:MountingHole_2.2mm_M2_ISO7380_Pad" (at 128.27 95.25 0)
+      (effects (font (size 1.27 1.27)) hide)
+    )
+    (property "Datasheet" "~" (at 128.27 95.25 0)
+      (effects (font (size 1.27 1.27)) hide)
+    )
+    (pin "1")
+    (instances
+      (project "YRM1001"
+        (path "/057aacfa-f1e4-4456-b429-057d9e3da096"
+          (reference "H2") (unit 1)
         )
       )
@@
     )
   )
+  (symbol (lib_id "Mechanical:MountingHole_Pad") (at 138.43 95.25 0) (unit 1)
+    (in_bom yes) (on_board yes) (dnp no)
+    (property "Reference" "H4" (at 137.16 90.17 0)
+      (effects (font (size 1.27 1.27)) (justify left))
+    )
+    (property "Value" "MountingHole_Pad" (at 129.54 100.33 0)
+      (effects (font (size 1.27 1.27)) (justify left) hide)
+    )
+    (property "Footprint" "MountingHole:MountingHole_2.2mm_M2_ISO7380_Pad" (at 138.43 95.25 0)
+      (effects (font (size 1.27 1.27)) hide)
+    )
+    (property "Datasheet" "~" (at 138.43 95.25 0)
+      (effects (font (size 1.27 1.27)) hide)
+    )
+    (pin "1")
+    (instances
+      (project "YRM1001"
+        (path "/057aacfa-f1e4-4456-b429-057d9e3da096"
+          (reference "H4") (unit 1)
+        )
+      )
+    )
+  )
   (symbol (lib_id "Device:C") (at 66.04 170.18 180) (unit 1)
     (in_bom yes) (on_board yes) (dnp no) (fields_autoplaced)
@@
         (path "/057aacfa-f1e4-4456-b429-057d9e3da096"
           (reference "#PWR05") (unit 1)
+        )
+      )
+      (project "UHF RFID board"
+        (path "/d8d0a45f-1f46-4ba4-9944-4b3c9d150d73"
+          (reference "#PWR08") (unit 1)
+        )
+      )
+    )
+  )
+  (symbol (lib_id "power:GND") (at 123.19 97.79 0) (mirror y) (unit 1)
+    (in_bom yes) (on_board yes) (dnp no)
+    (property "Reference" "#PWR014" (at 123.19 104.14 0)
+      (effects (font (size 1.27 1.27)) hide)
+    )
+    (property "Value" "GND" (at 123.19 101.6 90)
+      (effects (font (size 1.27 1.27)) (justify right))
+    )
+    (property "Footprint" "" (at 123.19 97.79 0)
+      (effects (font (size 1.27 1.27)) hide)
+    )
+    (property "Datasheet" "" (at 123.19 97.79 0)
+      (effects (font (size 1.27 1.27)) hide)
+    )
+    (pin "1")
+    (instances
+      (project "YRM1001"
+        (path "/057aacfa-f1e4-4456-b429-057d9e3da096"
+          (reference "#PWR014") (unit 1)
         )
       )
@@
         )
       )
+    )
+  )
+  (symbol (lib_id "Mechanical:MountingHole_Pad") (at 133.35 95.25 0) (unit 1)
+    (in_bom yes) (on_board yes) (dnp no)
+    (property "Reference" "H3" (at 132.08 90.17 0)
+      (effects (font (size 1.27 1.27)) (justify left))
+    )
+    (property "Value" "MountingHole_Pad" (at 124.46 100.33 0)
+      (effects (font (size 1.27 1.27)) (justify left) hide)
+    )
+    (property "Footprint" "MountingHole:MountingHole_2.2mm_M2_ISO7380_Pad" (at 133.35 95.25 0)
+      (effects (font (size 1.27 1.27)) hide)
+    )
+    (property "Datasheet" "~" (at 133.35 95.25 0)
+      (effects (font (size 1.27 1.27)) hide)
+    )
+    (pin "1")
+    (instances
+      (project "YRM1001"
+        (path "/057aacfa-f1e4-4456-b429-057d9e3da096"
+          (reference "H3") (unit 1)
+        )
+      )
+    )
+  )
+  (symbol (lib_id "Mechanical:MountingHole_Pad") (at 123.19 95.25 0) (unit 1)
+    (in_bom yes) (on_board yes) (dnp no)
+    (property "Reference" "H1" (at 121.92 90.17 0)
+      (effects (font (size 1.27 1.27)) (justify left))
+    )
+    (property "Value" "MountingHole_Pad" (at 118.11 100.33 0)
+      (effects (font (size 1.27 1.27)) (justify left) hide)
+    )
+    (property "Footprint" "MountingHole:MountingHole_2.2mm_M2_ISO7380_Pad" (at 123.19 95.25 0)
+      (effects (font (size 1.27 1.27)) hide)
+    )
+    (property "Datasheet" "~" (at 123.19 95.25 0)
+      (effects (font (size 1.27 1.27)) hide)
+    )
+    (pin "1")
+    (instances
+      (project "YRM1001"
+        (path "/057aacfa-f1e4-4456-b429-057d9e3da096"
+          (reference "H1") (unit 1)
+        )
+      )
